File: foc-board.kicad_pcb (KiCad board)
At the start: 4 copper layers, 70 x 70 mm, 143 parts, among them J1 , J2 USB_B_Mini, J3 Conn_01x02_Male, J4 Conn_01x02_Male, J5 Conn_01x01, J6 Conn_01x02_Male, J7 Conn_01x02, J8 Conn_01x01, J9 Conn_01x01, Q1 TK90S06N1L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

Commit message: add schem
Other:
- rule pad_to_mask_clearance: 0.05 -> 0.1
